File: ZynqBoard/PCB/ZynqBoard/AUDIO.sch (KiCad schematic (older format))
At the start: 20 parts, among them J5 35RAPC2BHN2, U11 AK4373EN, U12 PLT133_T10W, U13 PLR135_T10

Commit message: ZynqBoard PCB 設計完了
Parts:
- C135, C137, C139, C141, C143, C144, R67, R68, R69: 購入済み (none) -> -
- C136, C138, U12, U13: 購入済み (none) -> a
- C140, C142, J5, U11: 購入済み (none) -> d
- L10, L8, L9: footprint Inductors_SMD:L_0603 -> Inductors_SMD:L_0402; 購入済み (none) -> d
Changed lines of the file:
@@
 F 2 "Housings_DFN_QFN:QFN-32-1EP_5x5mm_Pitch0.5mm" H 5550 2650 50  0001 C CNN
 F 3 "" H 5550 2650 50  0001 C CNN
+F 4 "d" H 0   0   50  0001 C CNN "購入済み"
 	1    5550 2650
 	1    0    0    -1
@@
 F 2 "KiCad_Footprints:PLT133" H 8950 5800 50  0001 C CNN
 F 3 "" H 8950 5800 50  0001 C CNN
+F 4 "a" H 0   0   50  0001 C CNN "購入済み"
 	1    8950 5800
 	-1   0    0    -1
@@
 F 2 "KiCad_Footprints:PLT133" H 8950 5350 50  0001 C CNN
 F 3 "" H 8950 5350 50  0001 C CNN
+F 4 "a" H 0   0   50  0001 C CNN "購入済み"
 	1    8950 4950
 	1    0    0    -1
@@
 F 0 "L10" V 7425 5750 50  0000 L CNN
 F 1 "600ohm@100MHz" V 7200 5700 50  0000 C CNN
-F 2 "Inductors_SMD:L_0603" V 7280 5700 50  0001 C CNN
+F 2 "Inductors_SMD:L_0402" V 7280 5700 50  0001 C CNN
 F 3 "~" H 7350 5700 50  0001 C CNN
+F 4 "d" H 0   0   50  0001 C CNN "購入済み"
 	1    7350 5700
 	0    -1   -1   0
@@
 F 2 "Capacitors_SMD:C_0402_NoSilk" H 7800 5050 50  0001 C CNN
 F 3 "~" H 7800 5050 50  0001 C CNN
+F 4 "-" H 0   0   50  0001 C CNN "購入済み"
 	1    7800 5050
 	1    0    0    -1
@@
 F 2 "Capacitors_SMD:C_0402_NoSilk" H 7800 5900 50  0001 C CNN
 F 3 "~" H 7800 5900 50  0001 C CNN
+F 4 "-" H 0   0   50  0001 C CNN "購入済み"
 	1    7800 5900
 	1    0    0    -1
@@
 F 0 "L8" V 3325 1350 50  0000 L CNN
 F 1 "600ohm@100MHz" V 3100 1300 50  0000 C CNN
-F 2 "Inductors_SMD:L_0603" V 3180 1300 50  0001 C CNN
+F 2 "Inductors_SMD:L_0402" V 3180 1300 50  0001 C CNN
 F 3 "~" H 3250 1300 50  0001 C CNN
+F 4 "d" H 0   0   50  0001 C CNN "購入済み"
 	1    3250 1300
 	0    -1   -1   0
@@
 F 2 "Capacitors_SMD:C_0402_NoSilk" H 4000 1450 50  0001 C CNN
 F 3 "~" H 4000 1450 50  0001 C CNN
+F 4 "-" H 0   0   50  0001 C CNN "購入済み"
 	1    4000 1450
 	1    0    0    -1
@@
 F 2 "Capacitors_SMD:C_0603" H 3750 1450 50  0001 C CNN
 F 3 "~" H 3750 1450 50  0001 C CNN
+F 4 "a" H 0   0   50  0001 C CNN "購入済み"
 	1    3750 1450
 	1    0    0    -1
@@
 F 0 "L9" V 3325 1900 50  0000 L CNN
 F 1 "600ohm@100MHz" V 3100 1850 50  0000 C CNN
-F 2 "Inductors_SMD:L_0603" V 3180 1850 50  0001 C CNN
+F 2 "Inductors_SMD:L_0402" V 3180 1850 50  0001 C CNN
 F 3 "~" H 3250 1850 50  0001 C CNN
+F 4 "d" H 0   0   50  0001 C CNN "購入済み"
 	1    3250 1850
 	0    -1   -1   0
@@
 F 2 "Capacitors_SMD:C_0402_NoSilk" H 4000 2000 50  0001 C CNN
 F 3 "~" H 4000 2000 50  0001 C CNN
+F 4 "-" H 0   0   50  0001 C CNN "購入済み"
 	1    4000 2000
 	1    0    0    -1
@@
 F 2 "Capacitors_SMD:C_0603" H 3750 2000 50  0001 C CNN
 F 3 "~" H 3750 2000 50  0001 C CNN
+F 4 "a" H 0   0   50  0001 C CNN "購入済み"
 	1    3750 2000
 	1    0    0    -1
@@
 F 2 "Capacitors_SMD:C_0402_NoSilk" H 4850 1300 50  0001 C CNN
 F 3 "~" H 4850 1300 50  0001 C CNN
+F 4 "-" H 0   0   50  0001 C CNN "購入済み"
 	1    4850 1300
 	1    0    0    -1
@@
 F 2 "Capacitors_SMD:C_0402_NoSilk" H 6400 3700 50  0001 C CNN
 F 3 "~" H 6400 3700 50  0001 C CNN
+F 4 "-" H 0   0   50  0001 C CNN "購入済み"
 	1    6400 3700
 	1    0    0    -1
@@
 F 2 "Capacitors_SMD:C_0603" H 6650 3700 50  0001 C CNN
 F 3 "~" H 6650 3700 50  0001 C CNN
+F 4 "d" H 0   0   50  0001 C CNN "購入済み"
 	1    6650 3700
 	1    0    0    -1
@@
 F 2 "Capacitors_SMD:C_0402_NoSilk" H 7000 3500 50  0001 C CNN
 F 3 "~" H 7000 3500 50  0001 C CNN
+F 4 "d" H 0   0   50  0001 C CNN "購入済み"
 	1    7000 3500
 	1    0    0    -1
@@
 F 2 "Resistors_SMD:R_0603" V 3130 5050 50  0001 C CNN
 F 3 "~" H 3200 5050 50  0001 C CNN
+F 4 "-" H 0   0   50  0001 C CNN "購入済み"
 	1    3200 5050
 	1    0    0    -1
@@
 F 2 "Resistors_SMD:R_0603" V 3330 5050 50  0001 C CNN
 F 3 "~" H 3400 5050 50  0001 C CNN
+F 4 "-" H 0   0   50  0001 C CNN "購入済み"
 	1    3400 5050
 	1    0    0    -1
@@
 F 2 "Resistors_SMD:R_0603" V 3130 5750 50  0001 C CNN
 F 3 "~" H 3200 5750 50  0001 C CNN
+F 4 "-" H 0   0   50  0001 C CNN "購入済み"
 	1    3200 5750
 	1    0    0    -1
@@
 F 2 "KiCad_Footprints:35RAPC" H 8850 2750 50  0001 C CNN
 F 3 "" H 8850 2750 50  0001 C CNN
+F 4 "d" H 0   0   50  0001 C CNN "購入済み"
 	1    8900 2750
 	1    0    0    1
