File: ZynqBoard/PCB/ZynqBoard/Config.sch (KiCad schematic (older format))
At the start: 21 parts, among them J1 JTAG-HS3, SW1 Select_SD/JTAG, U1 XC7Z020-1CLG484C

Commit message: ZynqBoard PCB 設計完了
Parts:
- C82, C83, C84, D1, R10, R13, R14, R15, R16, R17, R18, R20, R8, R9: 購入済み (none) -> -
- J1: 購入済み (none) -> a
- O1, R19, SW1, U1: 購入済み (none) -> d
- R11, R12: footprint Resistors_SMD:R_0603 -> Resistors_SMD:R_0402_NoSilk; 購入済み (none) -> d
Connections:
- net labels removed: VBUS_0.5A, VBUS_1.5A, VBUS_3.0A
- wire segments 111 -> 108
- no-connect marks 4 -> 7
Other:
- note removed: "From USB"
Changed lines of the file:
@@
 F 2 "KiCad_Footprints:BGA-484_22x22_19.0x19.0mm" H 5550 4900 50  0001 C CNN
 F 3 "" H 5550 4900 50  0001 C CNN
+F 4 "d" H 0   0   50  0001 C CNN "購入済み"
 	1    5550 2300
 	1    0    0    -1
@@
 F 3 "~" H 1300 2650 50  0001 C CNN
 F 4 "2mm pitch" H 1450 2150 50  0000 C CNN "MEMO"
+F 5 "a" H 0   0   50  0001 C CNN "購入済み"
 	1    1300 2650
 	1    0    0    -1
@@
 F 2 "Resistors_SMD:R_0603" V 2480 2750 50  0001 C CNN
 F 3 "~" H 2550 2750 50  0001 C CNN
+F 4 "-" H 0   0   50  0001 C CNN "購入済み"
 	1    2550 2750
 	1    0    0    -1
@@
 F 2 "Capacitors_SMD:C_0402_NoSilk" H 4450 1750 50  0001 C CNN
 F 3 "~" H 4450 1750 50  0001 C CNN
+F 4 "-" H 0   0   50  0001 C CNN "購入済み"
 	1    4450 1750
 	1    0    0    -1
@@
 F 2 "Capacitors_SMD:C_0402_NoSilk" H 4450 2350 50  0001 C CNN
 F 3 "~" H 4450 2350 50  0001 C CNN
+F 4 "-" H 0   0   50  0001 C CNN "購入済み"
 	1    4450 2350
 	1    0    0    -1
@@
 F 0 "R12" V 7180 2900 50  0000 C CNN
 F 1 "4.7k" V 7100 2900 50  0000 C CNN
-F 2 "Resistors_SMD:R_0603" V 7030 2900 50  0001 C CNN
+F 2 "Resistors_SMD:R_0402_NoSilk" V 7030 2900 50  0001 C CNN
 F 3 "~" H 7100 2900 50  0001 C CNN
+F 4 "d" H 0   0   50  0001 C CNN "購入済み"
 	1    7100 2900
 	0    -1   -1   0
@@
 F 2 "KiCad_Footprints:BGA-484_22x22_19.0x19.0mm" H 5550 7400 50  0001 C CNN
 F 3 "" H 5550 7400 50  0001 C CNN
+F 4 "d" H 0   0   50  0001 C CNN "購入済み"
 	6    5550 4800
 	1    0    0    -1
@@
 F 2 "Resistors_SMD:R_0603" V 8880 4350 50  0001 C CNN
 F 3 "~" H 8950 4350 50  0001 C CNN
+F 4 "-" H 0   0   50  0001 C CNN "購入済み"
 	1    8950 4350
 	0    -1   -1   0
@@
 F 2 "Resistors_SMD:R_0603" V 8880 4550 50  0001 C CNN
 F 3 "~" H 8950 4550 50  0001 C CNN
+F 4 "-" H 0   0   50  0001 C CNN "購入済み"
 	1    8950 4550
 	0    -1   -1   0
@@
 F 2 "Resistors_SMD:R_0603" V 8880 4750 50  0001 C CNN
 F 3 "~" H 8950 4750 50  0001 C CNN
+F 4 "-" H 0   0   50  0001 C CNN "購入済み"
 	1    8950 4750
 	0    -1   -1   0
@@
 F 2 "Resistors_SMD:R_0603" V 8880 4950 50  0001 C CNN
 F 3 "~" H 8950 4950 50  0001 C CNN
+F 4 "-" H 0   0   50  0001 C CNN "購入済み"
 	1    8950 4950
 	0    -1   -1   0
@@
 F 2 "Resistors_SMD:R_0603" V 8880 3950 50  0001 C CNN
 F 3 "~" H 8950 3950 50  0001 C CNN
+F 4 "-" H 0   0   50  0001 C CNN "購入済み"
 	1    8950 3950
 	0    -1   -1   0
@@
 F 2 "Resistors_SMD:R_0603" V 8880 5600 50  0001 C CNN
 F 3 "~" H 8950 5600 50  0001 C CNN
+F 4 "-" H 0   0   50  0001 C CNN "購入済み"
 	1    8950 5600
 	0    -1   -1   0
@@
 F 2 "Resistors_SMD:R_0603" V 8880 5800 50  0001 C CNN
 F 3 "~" H 8950 5800 50  0001 C CNN
+F 4 "-" H 0   0   50  0001 C CNN "購入済み"
 	1    8950 5800
 	0    -1   -1   0
@@
 F 2 "Buttons_Switches_THT:SW_CuK_OS102011MA1QN1_SPDT_Angled" H 9750 5700 50  0001 C CNN
 F 3 "" H 9750 5700 50  0001 C CNN
+F 4 "d" H 0   0   50  0001 C CNN "購入済み"
 	1    9750 5700
 	1    0    0    -1
@@
 F 0 "R11" V 4580 2900 50  0000 C CNN
 F 1 "4.7k" V 4500 2900 50  0000 C CNN
-F 2 "Resistors_SMD:R_0603" V 4430 2900 50  0001 C CNN
+F 2 "Resistors_SMD:R_0402_NoSilk" V 4430 2900 50  0001 C CNN
 F 3 "~" H 4500 2900 50  0001 C CNN
+F 4 "d" H 0   0   50  0001 C CNN "購入済み"
 	1    4500 2900
 	0    -1   -1   0
@@
 F 2 "LEDs:LED_0603" H 9600 2500 50  0001 C CNN
 F 3 "~" H 9600 2500 50  0001 C CNN
+F 4 "-" H 0   0   50  0001 C CNN "購入済み"
 	1    9600 2500
 	0    -1   -1   0
@@
 F 2 "Resistors_SMD:R_0603" V 9530 1650 50  0001 C CNN
 F 3 "~" H 9600 1650 50  0001 C CNN
+F 4 "-" H 0   0   50  0001 C CNN "購入済み"
 	1    9600 1650
 	1    0    0    -1
@@
 F 2 "Resistors_SMD:R_0603" V 9530 2150 50  0001 C CNN
 F 3 "~" H 9600 2150 50  0001 C CNN
+F 4 "-" H 0   0   50  0001 C CNN "購入済み"
 	1    9600 2150
 	1    0    0    -1
@@
 F 2 "KiCad_Footprints:DSC1001_CDFN-4_3.2x2.5" H 2850 5650 60  0001 C CNN
 F 3 "" H 2850 5650 60  0001 C CNN
+F 4 "d" H 0   0   50  0001 C CNN "購入済み"
 	1    2850 5650
 	1    0    0    -1
@@
 F 2 "Capacitors_SMD:C_0402_NoSilk" H 1700 5500 50  0001 C CNN
 F 3 "~" H 1700 5500 50  0001 C CNN
+F 4 "-" H 0   0   50  0001 C CNN "購入済み"
 	1    1700 5500
 	1    0    0    -1
@@
 F 2 "Resistors_SMD:R_0603" V 3380 5650 50  0001 C CNN
 F 3 "~" H 3450 5650 50  0001 C CNN
+F 4 "d" H 0   0   50  0001 C CNN "購入済み"
 	1    3450 5650
 	0    -1   -1   0
@@
 Text GLabel 4150 1600 0    50   Input ~ 0
 XADC_1V8
-Text GLabel 6400 3900 2    50   Input ~ 0
-VBUS_0.5A
-Text GLabel 6400 4000 2    50   Input ~ 0
-VBUS_1.5A
-Text GLabel 6400 4100 2    50   Input ~ 0
-VBUS_3.0A
-Wire Wire Line
-	6400 4100 6250 4100
-Wire Wire Line
-	6250 4000 6400 4000
-Wire Wire Line
-	6400 3900 6250 3900
+Text GLabel 6400 4400 2    50   BiDi ~ 0
+HP_SCL
 Text GLabel 6400 4300 2    50   BiDi ~ 0
-HP_SCL
-Text GLabel 6400 4400 2    50   BiDi ~ 0
 HP_SDA
 Text GLabel 6400 4200 2    50   Output ~ 0
@@
 Wire Notes Line
 	6950 4450 6900 4450
-Wire Notes Line
-	6900 4125 6950 4125
-Wire Notes Line
-	6950 4125 6950 3850
-Wire Notes Line
-	6950 3850 6900 3850
 Text Notes 7000 4350 0    50   ~ 0
 To AUDIO
-Text Notes 7000 4050 0    50   ~ 0
-From USB
+NoConn ~ 6250 3900
+NoConn ~ 6250 4000
+NoConn ~ 6250 4100
 $EndSCHEMATC
