File: ZynqBoard/PCB/ZynqBoard/DDR.sch (KiCad schematic (older format))
At the start: 32 parts, among them U1 XC7Z020-1CLG484C, U2 IS43TR16256AL-125KBL

Commit message: ZynqBoard PCB 設計完了
Parts:
- C1, C10, C11, C12, C13, C14, C15, C16, C17, C18, C19, C2, C23, C4, C5, C6, C7, C8, C9, U1: 購入済み (none) -> d
- C20, C21, C22: 購入済み (none) -> a
- C3, R2: 購入済み (none) -> -
- R1: footprint Resistors_SMD:R_0603 -> Resistors_SMD:R_0402_NoSilk; 購入済み (none) -> d
- R3, R6, R7: Tolerance (none) -> 1%; 購入済み (none) -> d
- R4, R5: footprint Resistors_SMD:R_0603 -> Resistors_SMD:R_0402; 購入済み (none) -> d
- U2: footprint KiCad_Footprints:BGA-484_22x22_19.0x19.0mm -> KiCad_Footprints:BGA-96_2x3x16_9.0x13.0mm_Pitch0.8mm; 購入済み (none) -> d
Changed lines of the file:
@@
 F 0 "U2" H 8150 3250 50  0000 C CNN
 F 1 "IS43TR16256AL-125KBL" H 8150 3150 50  0000 C CNN
-F 2 "KiCad_Footprints:BGA-484_22x22_19.0x19.0mm" H 8150 3150 50  0001 C CNN
+F 2 "KiCad_Footprints:BGA-96_2x3x16_9.0x13.0mm_Pitch0.8mm" H 8150 3150 50  0001 C CNN
 F 3 "" H 8150 3150 50  0001 C CNN
+F 4 "d" H 0   0   50  0001 C CNN "購入済み"
 	1    8150 3150
 	1    0    0    -1
@@
 	3950 4000 4550 4000
 Wire Wire Line
+	1150 3500 1750 3500
+Wire Wire Line
+	1150 3900 1750 3900
+Wire Wire Line
+	1150 4100 1750 4100
+Wire Wire Line
+	1150 3600 1750 3600
+Wire Wire Line
+	1150 3700 1750 3700
+Wire Wire Line
+	1150 4200 1750 4200
+Wire Wire Line
+	1150 3800 1750 3800
+Wire Wire Line
+	1150 2700 1750 2700
+Wire Wire Line
+	1150 2900 1750 2900
+Wire Wire Line
+	1150 3200 1750 3200
+Wire Wire Line
+	1150 3300 1750 3300
+Wire Wire Line
+	1150 3000 1750 3000
+Wire Wire Line
 	1150 2800 1750 2800
 Wire Wire Line
-	1150 2900 1750 2900
-Wire Wire Line
-	1150 3000 1750 3000
-Wire Wire Line
 	1150 3100 1750 3100
 Wire Wire Line
-	1150 3200 1750 3200
-Wire Wire Line
-	1150 3300 1750 3300
-Wire Wire Line
 	1150 3400 1750 3400
 Wire Wire Line
-	1150 3500 1750 3500
-Wire Wire Line
-	1150 3600 1750 3600
-Wire Wire Line
-	1150 3700 1750 3700
-Wire Wire Line
-	1150 3800 1750 3800
-Wire Wire Line
-	1150 3900 1750 3900
-Wire Wire Line
 	1150 4000 1750 4000
 Wire Wire Line
-	1150 4100 1750 4100
-Wire Wire Line
-	1150 4200 1750 4200
-Wire Wire Line
-	1150 2700 1750 2700
+	1150 4800 1750 4800
 Wire Wire Line
 	1150 4700 1750 4700
 Wire Wire Line
-	1150 4800 1750 4800
+	1150 5600 1750 5600
+Wire Wire Line
+	1150 5700 1750 5700
 Wire Wire Line
 	1150 5400 1750 5400
 Wire Wire Line
 	1150 5500 1750 5500
-Wire Wire Line
-	1150 5600 1750 5600
-Wire Wire Line
-	1150 5700 1750 5700
 NoConn ~ 1750 5300
 NoConn ~ 1750 5200
@@
 Text Label 4550 2500 2    50   ~ 0
 DDR_A0
+Text Label 1150 3400 0    50   ~ 0
+DDR_DQ0
+Text Label 1150 3100 0    50   ~ 0
+DDR_DQ1
+Text Label 1150 2800 0    50   ~ 0
+DDR_DQ2
+Text Label 1150 3000 0    50   ~ 0
+DDR_DQ3
+Text Label 1150 3300 0    50   ~ 0
+DDR_DQ4
+Text Label 1150 3200 0    50   ~ 0
+DDR_DQ5
+Text Label 1150 2900 0    50   ~ 0
+DDR_DQ6
+Text Label 1150 2700 0    50   ~ 0
+DDR_DQ7
+Text Label 1150 3800 0    50   ~ 0
+DDR_DQ8
 Text Label 1150 4200 0    50   ~ 0
-DDR_DQ0
+DDR_DQ9
+Text Label 1150 3700 0    50   ~ 0
+DDR_DQ10
+Text Label 1150 3900 0    50   ~ 0
+DDR_DQ11
+Text Label 1150 3600 0    50   ~ 0
+DDR_DQ12
 Text Label 1150 4100 0    50   ~ 0
-DDR_DQ1
+DDR_DQ13
+Text Label 1150 3500 0    50   ~ 0
+DDR_DQ14
 Text Label 1150 4000 0    50   ~ 0
-DDR_DQ2
-Text Label 1150 3900 0    50   ~ 0
-DDR_DQ3
-Text Label 1150 3800 0    50   ~ 0
-DDR_DQ4
-Text Label 1150 3700 0    50   ~ 0
-DDR_DQ5
-Text Label 1150 3600 0    50   ~ 0
-DDR_DQ6
-Text Label 1150 3500 0    50   ~ 0
-DDR_DQ7
-Text Label 1150 3400 0    50   ~ 0
-DDR_DQ8
-Text Label 1150 3300 0    50   ~ 0
-DDR_DQ9
-Text Label 1150 3200 0    50   ~ 0
-DDR_DQ10
-Text Label 1150 3100 0    50   ~ 0
-DDR_DQ11
-Text Label 1150 3000 0    50   ~ 0
-DDR_DQ12
-Text Label 1150 2900 0    50   ~ 0
-DDR_DQ13
-Text Label 1150 2800 0    50   ~ 0
-DDR_DQ14
-Text Label 1150 2700 0    50   ~ 0
 DDR_DQ15
 Text Label 4550 3000 2    50   ~ 0
@@
 Text Label 4550 2800 2    50   ~ 0
 DDR_BA2
+Text Label 1150 4800 0    50   ~ 0
+DDR_DM1
 Text Label 1150 4700 0    50   ~ 0
-DDR_DM1
-Text Label 1150 4800 0    50   ~ 0
 DDR_DM0
+Text Label 1150 5600 0    50   ~ 0
+DDR_DQS_1_P
+Text Label 1150 5700 0    50   ~ 0
+DDR_DQS_1_N
 Text Label 1150 5400 0    50   ~ 0
-DDR_DQS_1_P
+DDR_DQS_0_P
 Text Label 1150 5500 0    50   ~ 0
-DDR_DQS_1_N
-Text Label 1150 5600 0    50   ~ 0
-DDR_DQS_0_P
-Text Label 1150 5700 0    50   ~ 0
 DDR_DQS_0_N
 Text Label 4550 3300 2    50   ~ 0
@@
 F 0 "R1" V 4280 4700 50  0000 C CNN
 F 1 "80" V 4200 4700 50  0000 C CNN
-F 2 "Resistors_SMD:R_0603" V 4130 4700 50  0001 C CNN
+F 2 "Resistors_SMD:R_0402_NoSilk" V 4130 4700 50  0001 C CNN
 F 3 "~" H 4200 4700 50  0001 C CNN
+F 4 "d" H 0   0   50  0001 C CNN "購入済み"
 	1    4200 4700
 	0    -1   -1   0
@@
 F 2 "Capacitors_SMD:C_0402_NoSilk" H 4450 5150 50  0001 C CNN
 F 3 "~" H 4450 5150 50  0001 C CNN
+F 4 "-" H 0   0   50  0001 C CNN "購入済み"
 	1    4450 5150
 	1    0    0    -1
@@
 F 0 "R4" V 4280 5500 50  0000 C CNN
 F 1 "80" V 4200 5500 50  0000 C CNN
-F 2 "Resistors_SMD:R_0603" V 4130 5500 50  0001 C CNN
+F 2 "Resistors_SMD:R_0402" V 4130 5500 50  0001 C CNN
 F 3 "~" H 4200 5500 50  0001 C CNN
+F 4 "d" H 0   0   50  0001 C CNN "購入済み"
 	1    4200 5500
 	0    -1   -1   0
@@
 F 0 "R5" V 4280 5700 50  0000 C CNN
 F 1 "80" V 4200 5700 50  0000 C CNN
-F 2 "Resistors_SMD:R_0603" V 4130 5700 50  0001 C CNN
+F 2 "Resistors_SMD:R_0402" V 4130 5700 50  0001 C CNN
 F 3 "~" H 4200 5700 50  0001 C CNN
+F 4 "d" H 0   0   50  0001 C CNN "購入済み"
 	1    4200 5700
 	0    -1   -1   0
@@
 F 3 "~" H 6300 1050 50  0001 C CNN
 F 4 "CA Byp" H 6100 1150 50  0000 C CNN "MEMO"
+F 5 "d" H 0   0   50  0001 C CNN "購入済み"
 	1    6300 1050
 	1    0    0    -1
@@
 F 3 "~" H 6300 1350 50  0001 C CNN
 F 4 "DQ Byp" H 6100 1300 50  0000 C CNN "MEMO"
+F 5 "d" H 0   0   50  0001 C CNN "購入済み"
 	1    6300 1350
 	1    0    0    -1
@@
 F 2 "Resistors_SMD:R_0603" V 10230 4950 50  0001 C CNN
 F 3 "~" H 10300 4950 50  0001 C CNN
+F 4 "1%" V 10200 4950 50  0000 C CNN "Tolerance"
+F 5 "d" H 0   0   50  0001 C CNN "購入済み"
 	1    10300 4950
 	1    0    0    -1
@@
 F 2 "Resistors_SMD:R_0603" V 9580 4950 50  0001 C CNN
 F 3 "~" H 9650 4950 50  0001 C CNN
+F 4 "-" H 0   0   50  0001 C CNN "購入済み"
 	1    9650 4950
 	1    0    0    -1
@@
 F 2 "Capacitors_SMD:C_0402_NoSilk" H 6000 6050 50  0001 C CNN
 F 3 "~" H 6000 6050 50  0001 C CNN
+F 4 "d" H 0   0   50  0001 C CNN "購入済み"
 	1    6000 6050
 	1    0    0    -1
@@
 F 2 "Capacitors_SMD:C_0402_NoSilk" H 6250 6050 50  0001 C CNN
 F 3 "~" H 6250 6050 50  0001 C CNN
+F 4 "d" H 0   0   50  0001 C CNN "購入済み"
 	1    6250 6050
 	1    0    0    -1
@@
 F 2 "Capacitors_SMD:C_0402_NoSilk" H 6500 6050 50  0001 C CNN
 F 3 "~" H 6500 6050 50  0001 C CNN
+F 4 "d" H 0   0   50  0001 C CNN "購入済み"
 	1    6500 6050
 	1    0    0    -1
@@
 F 2 "Capacitors_SMD:C_0402_NoSilk" H 6750 6050 50  0001 C CNN
 F 3 "~" H 6750 6050 50  0001 C CNN
+F 4 "d" H 0   0   50  0001 C CNN "購入済み"
 	1    6750 6050
 	1    0    0    -1
@@
 F 2 "Capacitors_SMD:C_0402_NoSilk" H 7000 6050 50  0001 C CNN
 F 3 "~" H 7000 6050 50  0001 C CNN
+F 4 "d" H 0   0   50  0001 C CNN "購入済み"
 	1    7000 6050
 	1    0    0    -1
@@
 F 2 "Capacitors_SMD:C_0402_NoSilk" H 7250 6050 50  0001 C CNN
 F 3 "~" H 7250 6050 50  0001 C CNN
+F 4 "d" H 0   0   50  0001 C CNN "購入済み"
 	1    7250 6050
 	1    0    0    -1
@@
 F 2 "Capacitors_SMD:C_0402_NoSilk" H 7500 6050 50  0001 C CNN
 F 3 "~" H 7500 6050 50  0001 C CNN
+F 4 "d" H 0   0   50  0001 C CNN "購入済み"
 	1    7500 6050
 	1    0    0    -1
@@
 F 2 "Capacitors_SMD:C_0402_NoSilk" H 7750 6050 50  0001 C CNN
 F 3 "~" H 7750 6050 50  0001 C CNN
+F 4 "d" H 0   0   50  0001 C CNN "購入済み"
 	1    7750 6050
 	1    0    0    -1
@@
 F 2 "Capacitors_SMD:C_0402_NoSilk" H 8300 6050 50  0001 C CNN
 F 3 "~" H 8300 6050 50  0001 C CNN
+F 4 "d" H 0   0   50  0001 C CNN "購入済み"
 	1    8300 6050
 	1    0    0    -1
@@
 F 2 "Capacitors_SMD:C_0402_NoSilk" H 8550 6050 50  0001 C CNN
 F 3 "~" H 8550 6050 50  0001 C CNN
+F 4 "d" H 0   0   50  0001 C CNN "購入済み"
 	1    8550 6050
 	1    0    0    -1
@@
 F 2 "Capacitors_SMD:C_0402_NoSilk" H 8800 6050 50  0001 C CNN
 F 3 "~" H 8800 6050 50  0001 C CNN
+F 4 "d" H 0   0   50  0001 C CNN "購入済み"
 	1    8800 6050
 	1    0    0    -1
@@
 F 2 "Capacitors_SMD:C_0402_NoSilk" H 9050 6050 50  0001 C CNN
 F 3 "~" H 9050 6050 50  0001 C CNN
+F 4 "d" H 0   0   50  0001 C CNN "購入済み"
 	1    9050 6050
 	1    0    0    -1
@@
 F 2 "Capacitors_SMD:C_0402_NoSilk" H 9300 6050 50  0001 C CNN
 F 3 "~" H 9300 6050 50  0001 C CNN
+F 4 "d" H 0   0   50  0001 C CNN "購入済み"
 	1    9300 6050
 	1    0    0    -1
@@
 F 2 "Capacitors_SMD:C_0402_NoSilk" H 9550 6050 50  0001 C CNN
 F 3 "~" H 9550 6050 50  0001 C CNN
+F 4 "d" H 0   0   50  0001 C CNN "購入済み"
 	1    9550 6050
 	1    0    0    -1
@@
 F 2 "Capacitors_SMD:C_0402_NoSilk" H 9800 6050 50  0001 C CNN
 F 3 "~" H 9800 6050 50  0001 C CNN
+F 4 "d" H 0   0   50  0001 C CNN "購入済み"
 	1    9800 6050
 	1    0    0    -1
@@
 F 2 "Capacitors_SMD:C_0402_NoSilk" H 10050 6050 50  0001 C CNN
 F 3 "~" H 10050 6050 50  0001 C CNN
+F 4 "d" H 0   0   50  0001 C CNN "購入済み"
 	1    10050 6050
 	1    0    0    -1
@@
 F 2 "Capacitors_SMD:C_0402_NoSilk" H 6000 6950 50  0001 C CNN
 F 3 "~" H 6000 6950 50  0001 C CNN
+F 4 "a" H 0   0   50  0001 C CNN "購入済み"
 	1    6000 6950
 	1    0    0    -1
@@
 F 2 "Capacitors_SMD:C_0402_NoSilk" H 6300 6950 50  0001 C CNN
 F 3 "~" H 6300 6950 50  0001 C CNN
+F 4 "a" H 0   0   50  0001 C CNN "購入済み"
 	1    6300 6950
 	1    0    0    -1
@@
 F 2 "Capacitors_SMD:C_0603" H 6600 6950 50  0001 C CNN
 F 3 "~" H 6600 6950 50  0001 C CNN
+F 4 "a" H 0   0   50  0001 C CNN "購入済み"
 	1    6600 6950
 	1    0    0    -1
@@
 F 2 "Resistors_SMD:R_0603" V 1480 6650 50  0001 C CNN
 F 3 "~" H 1550 6650 50  0001 C CNN
+F 4 "1%" V 1450 6650 50  0000 C CNN "Tolerance"
+F 5 "d" V 1550 6650 50  0001 C CNN "購入済み"
 	1    1550 6650
 	1    0    0    -1
@@
 F 2 "Resistors_SMD:R_0603" V 1480 7050 50  0001 C CNN
 F 3 "~" H 1550 7050 50  0001 C CNN
+F 4 "1%" V 1450 7050 50  0000 C CNN "Tolerance"
+F 5 "d" H 0   0   50  0001 C CNN "購入済み"
 	1    1550 7050
 	1    0    0    -1
@@
 F 2 "Capacitors_SMD:C_0402_NoSilk" H 1900 7050 50  0001 C CNN
 F 3 "~" H 1900 7050 50  0001 C CNN
+F 4 "d" H 0   0   50  0001 C CNN "購入済み"
 	1    1900 7050
 	1    0    0    -1
@@
 F 2 "KiCad_Footprints:BGA-484_22x22_19.0x19.0mm" H 2850 6100 50  0001 C CNN
 F 3 "" H 2850 6100 50  0001 C CNN
+F 4 "d" H 0   0   50  0001 C CNN "購入済み"
 	4    2850 3500
 	1    0    0    -1
