File: ZynqBoard/PCB/ZynqBoard/I_F.sch (KiCad schematic (older format))
At the start: 30 parts, among them P1 Universal I/F 1, P2 Universal I/F 2, P3 Universal I/F 3, P4 Universal I/F 4, P5 Universal I/F 5, P6 Universal I/F 6, Q3 IRLML6344TRPbF, Q4 IRLML6344TRPbF, Q5 IRLML6344TRPbF, Q6 IRLML6344TRPbF, Q7 IRLML6344TRPbF, Q8 IRLML6344TRPbF, U14 M74HC365, U15 M74HC365, U16 M74HC365, U17 M74HC365, U18 M74HC365, U19 M74HC365

Commit message: ZynqBoard PCB 設計完了
Parts:
- C145, C146, C147, C148, C149, C150, P1, P2, P3, P4, P5, P6, R70, R71, R72, R73, R74, R75: 購入済み (none) -> -
- Q3, Q4, Q5, Q6, Q7, Q8: 購入済み (none) -> a
- U14, U15, U16, U17, U18, U19: 購入済み (none) -> d
Changed lines of the file:
@@
 F 2 "Pin_Headers:Pin_Header_Straight_2x05_Pitch2.54mm" H 8400 1650 50  0001 C CNN
 F 3 "" H 8400 1650 50  0001 C CNN
+F 4 "-" H 0   0   50  0001 C CNN "購入済み"
 	1    8450 1650
 	1    0    0    -1
@@
 F 2 "TO_SOT_Packages_SMD:SOT-23" H 7850 2200 50  0001 C CNN
 F 3 "~" H 7650 2100 50  0001 C CNN
+F 4 "a" H 0   0   50  0001 C CNN "購入済み"
 	1    7650 2100
 	1    0    0    -1
@@
 F 2 "Resistors_SMD:R_0603" V 7180 2100 50  0001 C CNN
 F 3 "~" H 7250 2100 50  0001 C CNN
+F 4 "-" H 0   0   50  0001 C CNN "購入済み"
 	1    7250 2100
 	0    -1   -1   0
@@
 F 2 "Housings_SSOP:TSSOP-16_4.4x5mm_Pitch0.65mm" H 2050 2050 50  0001 C CNN
 F 3 "http://www.ti.com/lit/gpn/sn74LS365" H 2050 2050 50  0001 C CNN
+F 4 "d" H 0   0   50  0001 C CNN "購入済み"
 	1    2050 2050
 	1    0    0    -1
@@
 F 2 "Capacitors_SMD:C_0402_NoSilk" H 2250 1200 50  0001 C CNN
 F 3 "~" H 2250 1200 50  0001 C CNN
+F 4 "-" H 0   0   50  0001 C CNN "購入済み"
 	1    2250 1200
 	1    0    0    -1
@@
 Wire Wire Line
 	2550 2150 2900 2150
-Text Label 1200 1650 0    50   ~ 0
+Text Label 1200 1850 0    50   ~ 0
 1_SSCK
-Text GLabel 2950 1650 2    50   Output ~ 0
+Text GLabel 2950 1850 2    50   Output ~ 0
 IF1_SSCK
 Text Label 2900 1750 2    50   ~ 0
@@
 Text GLabel 1150 1750 0    50   Input ~ 0
 IF1_SRXD
-Text Label 1200 1850 0    50   ~ 0
+Text Label 1200 1650 0    50   ~ 0
 1_STXD
-Text GLabel 2950 1850 2    50   Output ~ 0
+Text GLabel 2950 1650 2    50   Output ~ 0
 IF1_STXD
 Text Label 2900 1950 2    50   ~ 0
@@
 F 2 "Pin_Headers:Pin_Header_Straight_2x05_Pitch2.54mm" H 10550 1650 50  0001 C CNN
 F 3 "" H 10550 1650 50  0001 C CNN
+F 4 "-" H 0   0   50  0001 C CNN "購入済み"
 	1    10600 1650
 	1    0    0    -1
@@
 F 2 "TO_SOT_Packages_SMD:SOT-23" H 10000 2200 50  0001 C CNN
 F 3 "~" H 9800 2100 50  0001 C CNN
+F 4 "a" H 0   0   50  0001 C CNN "購入済み"
 	1    9800 2100
 	1    0    0    -1
@@
 F 2 "Resistors_SMD:R_0603" V 9330 2100 50  0001 C CNN
 F 3 "~" H 9400 2100 50  0001 C CNN
+F 4 "-" H 0   0   50  0001 C CNN "購入済み"
 	1    9400 2100
 	0    -1   -1   0
@@
 F 2 "Pin_Headers:Pin_Header_Straight_2x05_Pitch2.54mm" H 8400 3500 50  0001 C CNN
 F 3 "" H 8400 3500 50  0001 C CNN
+F 4 "-" H 0   0   50  0001 C CNN "購入済み"
 	1    8450 3500
 	1    0    0    -1
@@
 F 2 "TO_SOT_Packages_SMD:SOT-23" H 7850 4050 50  0001 C CNN
 F 3 "~" H 7650 3950 50  0001 C CNN
+F 4 "a" H 0   0   50  0001 C CNN "購入済み"
 	1    7650 3950
 	1    0    0    -1
@@
 F 2 "Resistors_SMD:R_0603" V 7180 3950 50  0001 C CNN
 F 3 "~" H 7250 3950 50  0001 C CNN
+F 4 "-" H 0   0   50  0001 C CNN "購入済み"
 	1    7250 3950
 	0    -1   -1   0
@@
 F 2 "Pin_Headers:Pin_Header_Straight_2x05_Pitch2.54mm" H 10550 3500 50  0001 C CNN
 F 3 "" H 10550 3500 50  0001 C CNN
+F 4 "-" H 0   0   50  0001 C CNN "購入済み"
 	1    10600 3500
 	1    0    0    -1
@@
 F 2 "TO_SOT_Packages_SMD:SOT-23" H 10000 4050 50  0001 C CNN
 F 3 "~" H 9800 3950 50  0001 C CNN
+F 4 "a" H 0   0   50  0001 C CNN "購入済み"
 	1    9800 3950
 	1    0    0    -1
@@
 F 2 "Resistors_SMD:R_0603" V 9330 3950 50  0001 C CNN
 F 3 "~" H 9400 3950 50  0001 C CNN
+F 4 "-" H 0   0   50  0001 C CNN "購入済み"
 	1    9400 3950
 	0    -1   -1   0
@@
 F 2 "Pin_Headers:Pin_Header_Straight_2x05_Pitch2.54mm" H 8400 5300 50  0001 C CNN
 F 3 "" H 8400 5300 50  0001 C CNN
+F 4 "-" H 0   0   50  0001 C CNN "購入済み"
 	1    8450 5300
 	1    0    0    -1
@@
 F 2 "TO_SOT_Packages_SMD:SOT-23" H 7850 5850 50  0001 C CNN
 F 3 "~" H 7650 5750 50  0001 C CNN
+F 4 "a" H 0   0   50  0001 C CNN "購入済み"
 	1    7650 5750
 	1    0    0    -1
@@
 F 2 "Resistors_SMD:R_0603" V 7180 5750 50  0001 C CNN
 F 3 "~" H 7250 5750 50  0001 C CNN
+F 4 "-" H 0   0   50  0001 C CNN "購入済み"
 	1    7250 5750
 	0    -1   -1   0
@@
 F 2 "Pin_Headers:Pin_Header_Straight_2x05_Pitch2.54mm" H 10550 5300 50  0001 C CNN
 F 3 "" H 10550 5300 50  0001 C CNN
+F 4 "-" H 0   0   50  0001 C CNN "購入済み"
 	1    10600 5300
 	1    0    0    -1
@@
 F 2 "TO_SOT_Packages_SMD:SOT-23" H 10000 5850 50  0001 C CNN
 F 3 "~" H 9800 5750 50  0001 C CNN
+F 4 "a" H 0   0   50  0001 C CNN "購入済み"
 	1    9800 5750
 	1    0    0    -1
@@
 F 2 "Resistors_SMD:R_0603" V 9330 5750 50  0001 C CNN
 F 3 "~" H 9400 5750 50  0001 C CNN
+F 4 "-" H 0   0   50  0001 C CNN "購入済み"
 	1    9400 5750
 	0    -1   -1   0
@@
 F 2 "Housings_SSOP:TSSOP-16_4.4x5mm_Pitch0.65mm" H 4800 2050 50  0001 C CNN
 F 3 "http://www.ti.com/lit/gpn/sn74LS365" H 4800 2050 50  0001 C CNN
+F 4 "d" H 0   0   50  0001 C CNN "購入済み"
 	1    4800 2050
 	1    0    0    -1
@@
 F 2 "Capacitors_SMD:C_0402_NoSilk" H 5000 1200 50  0001 C CNN
 F 3 "~" H 5000 1200 50  0001 C CNN
+F 4 "-" H 0   0   50  0001 C CNN "購入済み"
 	1    5000 1200
 	1    0    0    -1
@@
 Wire Wire Line
 	5300 2150 5650 2150
-Text Label 3950 1650 0    50   ~ 0
+Text Label 3950 1850 0    50   ~ 0
 2_SSCK
-Text GLabel 5700 1650 2    50   Output ~ 0
+Text GLabel 5700 1850 2    50   Output ~ 0
 IF2_SSCK
 Text Label 5650 1750 2    50   ~ 0
@@
 Text GLabel 3900 1750 0    50   Input ~ 0
 IF2_SRXD
-Text Label 3950 1850 0    50   ~ 0
+Text Label 3950 1650 0    50   ~ 0
 2_STXD
-Text GLabel 5700 1850 2    50   Output ~ 0
+Text GLabel 5700 1650 2    50   Output ~ 0
 IF2_STXD
 Text Label 5650 1950 2    50   ~ 0
@@
 F 2 "Housings_SSOP:TSSOP-16_4.4x5mm_Pitch0.65mm" H 2050 4300 50  0001 C CNN
 F 3 "http://www.ti.com/lit/gpn/sn74LS365" H 2050 4300 50  0001 C CNN
+F 4 "d" H 0   0   50  0001 C CNN "購入済み"
 	1    2050 4300
 	1    0    0    -1
@@
 F 2 "Capacitors_SMD:C_0402_NoSilk" H 2250 3450 50  0001 C CNN
 F 3 "~" H 2250 3450 50  0001 C CNN
+F 4 "-" H 0   0   50  0001 C CNN "購入済み"
 	1    2250 3450
 	1    0    0    -1
@@
 Wire Wire Line
 	2550 4400 2900 4400
-Text Label 1200 3900 0    50   ~ 0
+Text Label 1200 4100 0    50   ~ 0
 3_SSCK
-Text GLabel 2950 3900 2    50   Output ~ 0
+Text GLabel 2950 4100 2    50   Output ~ 0
 IF3_SSCK
 Text Label 2900 4000 2    50   ~ 0
@@
 Text GLabel 1150 4000 0    50   Input ~ 0
 IF3_SRXD
-Text Label 1200 4100 0    50   ~ 0
+Text Label 1200 3900 0    50   ~ 0
 3_STXD
-Text GLabel 2950 4100 2    50   Output ~ 0
+Text GLabel 2950 3900 2    50   Output ~ 0
 IF3_STXD
 Text Label 2900 4200 2    50   ~ 0
@@
 F 2 "Housings_SSOP:TSSOP-16_4.4x5mm_Pitch0.65mm" H 4800 4300 50  0001 C CNN
 F 3 "http://www.ti.com/lit/gpn/sn74LS365" H 4800 4300 50  0001 C CNN
+F 4 "d" H 0   0   50  0001 C CNN "購入済み"
 	1    4800 4300
 	1    0    0    -1
@@
 F 2 "Capacitors_SMD:C_0402_NoSilk" H 5000 3450 50  0001 C CNN
 F 3 "~" H 5000 3450 50  0001 C CNN
+F 4 "-" H 0   0   50  0001 C CNN "購入済み"
 	1    5000 3450
 	1    0    0    -1
@@
 Text GLabel 5700 4100 2    50   Output ~ 0
 IF4_STXD
-Text Label 5650 4200 2    50   ~ 0
+Text Label 5650 4400 2    50   ~ 0
 4_HSCK
-Text GLabel 3900 4200 0    50   Input ~ 0
+Text GLabel 3900 4400 0    50   Input ~ 0
 IF4_HSCK
 Text Label 3950 4300 0    50   ~ 0
@@
 Text GLabel 5700 4300 2    50   Output ~ 0
 IF4_HRXD
-Text Label 5650 4400 2    50   ~ 0
+Text Label 5650 4200 2    50   ~ 0
 4_HTXD
-Text GLabel 3900 4400 0    50   Input ~ 0
+Text GLabel 3900 4200 0    50   Input ~ 0
 IF4_HTXD
 Wire Wire Line
@@
 F 2 "Housings_SSOP:TSSOP-16_4.4x5mm_Pitch0.65mm" H 2050 6550 50  0001 C CNN
 F 3 "http://www.ti.com/lit/gpn/sn74LS365" H 2050 6550 50  0001 C CNN
+F 4 "d" H 0   0   50  0001 C CNN "購入済み"
 	1    2050 6550
 	1    0    0    -1
@@
 F 2 "Capacitors_SMD:C_0402_NoSilk" H 2250 5700 50  0001 C CNN
 F 3 "~" H 2250 5700 50  0001 C CNN
+F 4 "-" H 0   0   50  0001 C CNN "購入済み"
 	1    2250 5700
 	1    0    0    -1
@@
 Text GLabel 2950 6350 2    50   Output ~ 0
 IF5_STXD
-Text Label 2900 6450 2    50   ~ 0
+Text Label 2900 6650 2    50   ~ 0
 5_HSCK
-Text GLabel 1150 6450 0    50   Input ~ 0
+Text GLabel 1150 6650 0    50   Input ~ 0
 IF5_HSCK
 Text Label 1200 6550 0    50   ~ 0
@@
 Text GLabel 2950 6550 2    50   Output ~ 0
 IF5_HRXD
-Text Label 2900 6650 2    50   ~ 0
+Text Label 2900 6450 2    50   ~ 0
 5_HTXD
-Text GLabel 1150 6650 0    50   Input ~ 0
+Text GLabel 1150 6450 0    50   Input ~ 0
 IF5_HTXD
 Wire Wire Line
@@
 F 2 "Housings_SSOP:TSSOP-16_4.4x5mm_Pitch0.65mm" H 4800 6550 50  0001 C CNN
 F 3 "http://www.ti.com/lit/gpn/sn74LS365" H 4800 6550 50  0001 C CNN
+F 4 "d" H 0   0   50  0001 C CNN "購入済み"
 	1    4800 6550
 	1    0    0    -1
@@
 F 2 "Capacitors_SMD:C_0402_NoSilk" H 5000 5700 50  0001 C CNN
 F 3 "~" H 5000 5700 50  0001 C CNN
+F 4 "-" H 0   0   50  0001 C CNN "購入済み"
 	1    5000 5700
 	1    0    0    -1
@@
 Wire Wire Line
 	5300 6650 5650 6650
-Text Label 3950 6150 0    50   ~ 0
+Text Label 3950 6350 0    50   ~ 0
 6_SSCK
-Text GLabel 5700 6150 2    50   Output ~ 0
+Text GLabel 5700 6350 2    50   Output ~ 0
 IF6_SSCK
 Text Label 5650 6250 2    50   ~ 0
@@
 Text GLabel 3900 6250 0    50   Input ~ 0
 IF6_SRXD
-Text Label 3950 6350 0    50   ~ 0
+Text Label 3950 6150 0    50   ~ 0
 6_STXD
-Text GLabel 5700 6350 2    50   Output ~ 0
+Text GLabel 5700 6150 2    50   Output ~ 0
 IF6_STXD
 Text Label 5650 6450 2    50   ~ 0
