File: ZynqBoard/PCB/ZynqBoard/PL_IO.sch (KiCad schematic (older format))
At the start: 5 parts, among them U1 XC7Z020-1CLG484C

Commit message: ZynqBoard PCB 設計完了
Parts:
- added TP1: TEST1, Measurement_Points:Measurement_Point_Round-SMD-Pad_Small, symbol Connector:TestPoint_Alt
- added TP2: TEST2, Measurement_Points:Measurement_Point_Round-SMD-Pad_Small, symbol Connector:TestPoint_Alt
- added TP3: TEST3, Measurement_Points:Measurement_Point_Round-SMD-Pad_Small, symbol Connector:TestPoint_Alt
- added TP4: TEST4, Measurement_Points:Measurement_Point_Round-SMD-Pad_Small, symbol Connector:TestPoint_Alt
- added unit 10 of U1
- D4, U1: 購入済み (none) -> d
- R76, R77, R78: 購入済み (none) -> -
Connections:
- net labels added: TEST1, TEST2, TEST3, TEST4, USB_RSTN
- wire segments 11 -> 19
- no-connect marks 0 -> 126
