File: ZynqBoard/PCB/ZynqBoard/PowerSupply.sch (KiCad schematic (older format))
At the start: 67 parts, among them Q1 FDS9926A, SW2 SW_SPDT, U4 ADP5052ACPZ-R7, U5 TPS25940ARVC, U6 ADP124ARHZ-3.3-R7, U7 REF3012

Commit message: ZynqBoard PCB 設計完了
Parts:
- C100, C104, C106, C111, C115, C116, C119, C120, C93, R28, R34, R37, R40, R41, R44, R47, R50: 購入済み (none) -> -
- C101, C102, C103, C105, C107, C109, C110, C113, C118, C94, C96, C97, C98, C99, L2, L3, L4, L5, Q1, R26, R27, R29, R30, R31, R32, R33, R35, R36, R38, R39, R42, R43, R45, R46, R49, SW2, U4, U5, U6, U7: 購入済み (none) -> d
- C108, C112, C114, C117, C89, C90, C91, C92, C95: 購入済み (none) -> a
- R48: value 4.7k -> 20k; MEMO NF -> (none); 購入済み (none) -> -
