File: ZynqBoard/PCB/ZynqBoard/SD.sch (KiCad schematic (older format))
At the start: 12 parts, among them J2 Hirose_DM3AT, U1 XC7Z020-1CLG484C, U3 TXS02612RTWR

Commit message: ZynqBoard PCB 設計完了
Parts:
- C85, C86, C87, R22: 購入済み (none) -> -
- C88, J2, R23, U1, U3: 購入済み (none) -> d
- R21, R24, R25: footprint Resistors_SMD:R_0603 -> Resistors_SMD:R_0402_NoSilk; Tolerance (none) -> 1%; 購入済み (none) -> d
Connections:
- net labels added: VBUS_0.5A, VBUS_1.5A, VBUS_3.0A
- wire segments 75 -> 78
- no-connect marks 37 -> 34
Other:
- note added: "From USB"
Changed lines of the file:
@@
 F 2 "Connectors_Card:Hirose_DM3AT-SF-PEJM5" H 10950 4150 50  0001 C CNN
 F 3 "https://www.hirose.com/product/en/download_file/key_name/DM3/category/Catalog/doc_file_id/49662/?file_category_id=4&item_id=195&is_series=1" H 8900 3550 50  0001 C CNN
+F 4 "d" H 0   0   50  0001 C CNN "購入済み"
 	1    8900 3450
 	1    0    0    -1
@@
 F 2 "Housings_DFN_QFN:QFN-24-1EP_4x4mm_Pitch0.5mm" H 6100 3550 50  0001 C CNN
 F 3 "" H 6100 3550 50  0001 C CNN
+F 4 "d" H 0   0   50  0001 C CNN "購入済み"
 	1    6100 3550
 	1    0    0    -1
@@
 F 2 "Resistors_SMD:R_0603" V 5380 3950 50  0001 C CNN
 F 3 "~" H 5450 3950 50  0001 C CNN
+F 4 "-" H 0   0   50  0001 C CNN "購入済み"
 	1    5450 3950
 	1    0    0    -1
@@
 F 2 "Resistors_SMD:R_0603" V 7330 4500 50  0001 C CNN
 F 3 "~" H 7400 4500 50  0001 C CNN
+F 4 "d" H 0   0   50  0001 C CNN "購入済み"
 	1    7400 4500
 	1    0    0    -1
@@
 F 2 "Capacitors_SMD:C_0402_NoSilk" H 8000 2500 50  0001 C CNN
 F 3 "~" H 8000 2500 50  0001 C CNN
+F 4 "-" H 0   0   50  0001 C CNN "購入済み"
 	1    8000 2500
 	1    0    0    -1
@@
 F 2 "Capacitors_SMD:C_0402_NoSilk" H 6900 2500 50  0001 C CNN
 F 3 "~" H 6900 2500 50  0001 C CNN
+F 4 "-" H 0   0   50  0001 C CNN "購入済み"
 	1    6900 2500
 	1    0    0    -1
@@
 F 2 "Capacitors_SMD:C_0402_NoSilk" H 5200 2500 50  0001 C CNN
 F 3 "~" H 5200 2500 50  0001 C CNN
+F 4 "-" H 0   0   50  0001 C CNN "購入済み"
 	1    5200 2500
 	1    0    0    -1
@@
 F 2 "KiCad_Footprints:BGA-484_22x22_19.0x19.0mm" H 2350 6750 50  0001 C CNN
 F 3 "" H 2350 6750 50  0001 C CNN
+F 4 "d" H 0   0   50  0001 C CNN "購入済み"
 	5    2350 4150
 	1    0    0    -1
@@
 	3550 2850 3050 2850
 Wire Wire Line
-	3050 2750 3550 2750
-Text Label 3550 2750 2    50   ~ 0
+	3050 2650 3550 2650
+Text Label 3550 2650 2    50   ~ 0
 SD_CD
 Text Label 3550 2850 2    50   ~ 0
@@
 F 0 "R21" V 3380 3350 50  0000 C CNN
 F 1 "40.2" V 3300 3350 50  0000 C CNN
-F 2 "Resistors_SMD:R_0603" V 3230 3350 50  0001 C CNN
+F 2 "Resistors_SMD:R_0402_NoSilk" V 3230 3350 50  0001 C CNN
 F 3 "~" H 3300 3350 50  0001 C CNN
+F 4 "1%" V 3375 3525 50  0000 C CNN "Tolerance"
+F 5 "d" H 0   0   50  0001 C CNN "購入済み"
 	1    3300 3350
 	0    1    1    0
@@
 F 0 "R24" V 5230 6250 50  0000 C CNN
 F 1 "10k" V 5150 6250 50  0000 C CNN
-F 2 "Resistors_SMD:R_0603" V 5080 6250 50  0001 C CNN
+F 2 "Resistors_SMD:R_0402_NoSilk" V 5080 6250 50  0001 C CNN
 F 3 "~" H 5150 6250 50  0001 C CNN
+F 4 "1%" V 5050 6250 50  0000 C CNN "Tolerance"
+F 5 "d" H 0   0   50  0001 C CNN "購入済み"
 	1    5150 6250
 	1    0    0    -1
@@
 F 0 "R25" V 5230 6650 50  0000 C CNN
 F 1 "10k" V 5150 6650 50  0000 C CNN
-F 2 "Resistors_SMD:R_0603" V 5080 6650 50  0001 C CNN
+F 2 "Resistors_SMD:R_0402_NoSilk" V 5080 6650 50  0001 C CNN
 F 3 "~" H 5150 6650 50  0001 C CNN
+F 4 "1%" V 5050 6650 50  0000 C CNN "Tolerance"
+F 5 "d" H 0   0   50  0001 C CNN "購入済み"
 	1    5150 6650
 	1    0    0    -1
@@
 F 2 "Capacitors_SMD:C_0402_NoSilk" H 5400 6650 50  0001 C CNN
 F 3 "~" H 5400 6650 50  0001 C CNN
+F 4 "d" H 0   0   50  0001 C CNN "購入済み"
 	1    5400 6650
 	1    0    0    -1
@@
 NoConn ~ 3050 2450
 NoConn ~ 3050 2550
-NoConn ~ 3050 2650
 NoConn ~ 3050 3450
 NoConn ~ 3050 3550
@@
 NoConn ~ 3050 4350
 NoConn ~ 3050 4450
-NoConn ~ 3050 4550
 NoConn ~ 3050 4650
-NoConn ~ 3050 4750
 NoConn ~ 3050 4850
 NoConn ~ 3050 4950
 NoConn ~ 3050 5050
-NoConn ~ 3050 5150
 NoConn ~ 3050 5250
 NoConn ~ 3050 5350
@@
 Text GLabel 3150 6150 2    50   BiDi ~ 0
 PS_SRST_B
+Wire Wire Line
+	3050 4550 3250 4550
+Wire Wire Line
+	3050 4750 3250 4750
+Wire Wire Line
+	3050 5150 3250 5150
+Text GLabel 3250 4550 2    50   Input ~ 0
+VBUS_0.5A
+Text GLabel 3250 4750 2    50   Input ~ 0
+VBUS_1.5A
+Text GLabel 3250 5150 2    50   Input ~ 0
+VBUS_3.0A
+Wire Notes Line
+	3750 5150 3800 5150
+Wire Notes Line
+	3800 5150 3800 4550
+Wire Notes Line
+	3800 4550 3750 4550
+Text Notes 3850 4875 0    50   ~ 0
+From USB
+NoConn ~ 3050 2750
 $EndSCHEMATC
