File: ZynqBoard/PCB/ZynqBoard/USB.sch (KiCad schematic (older format))
At the start: 41 parts, among them J3 Battery, J4 USB_C_Receptacle, Q2 Si2369DS, U10 93LC56BT-I_OTCT, U8 UTC2000, U9 FT-232H

Commit message: ZynqBoard PCB 設計完了
Parts:
- C121, J4, O2, Q2, R51, R56, R61, R62, R64, U10, U8: 購入済み (none) -> d
- C122, C123, C124, C126, C127, C128, C130, C131, C132, C133, C134, D2, D3, R52, R53, R54, R55, R57, R58, R59, R60, R63, R65, R66: 購入済み (none) -> -
- C125, C129, J3, U9: 購入済み (none) -> a
- L6, L7: footprint Inductors_SMD:L_0603 -> Inductors_SMD:L_0402; 購入済み (none) -> d
Connections:
- net labels added: +1V8
- net labels removed: +3V3
Changed lines of the file:
@@
 F 2 "Housings_DFN_QFN:QFN-16-1EP_3x3mm_Pitch0.5mm" H 5600 2650 50  0001 C CNN
 F 3 "" H 5600 2650 50  0001 C CNN
+F 4 "d" H 0   0   50  0001 C CNN "購入済み"
 	1    5600 2100
 	1    0    0    -1
@@
 F 2 "KiCad_Footprints:CX70M-24P1" H 1800 2300 50  0001 C CNN
 F 3 "http://www.usb.org/developers/docs/usb_31_033017.zip" H 1800 2300 50  0001 C CNN
+F 4 "d" H 0   0   50  0001 C CNN "購入済み"
 	1    1650 2300
 	1    0    0    -1
@@
 F 2 "TO_SOT_Packages_SMD:SOT-23" H 8150 1200 50  0001 C CNN
 F 3 "~" H 7950 1100 50  0001 C CNN
+F 4 "d" H 0   0   50  0001 C CNN "購入済み"
 	1    7950 1100
 	0    1    -1   0
@@
 F 2 "Resistors_SMD:R_0603" V 2480 3500 50  0001 C CNN
 F 3 "~" H 2550 3500 50  0001 C CNN
+F 4 "d" H 0   0   50  0001 C CNN "購入済み"
 	1    2550 3500
 	1    0    0    -1
@@
 F 2 "Resistors_SMD:R_0603" V 2680 3500 50  0001 C CNN
 F 3 "~" H 2750 3500 50  0001 C CNN
+F 4 "d" H 0   0   50  0001 C CNN "購入済み"
 	1    2750 3500
 	1    0    0    -1
@@
 F 2 "Resistors_SMD:R_0603" V 2980 3200 50  0001 C CNN
 F 3 "~" H 3050 3200 50  0001 C CNN
+F 4 "-" H 0   0   50  0001 C CNN "購入済み"
 	1    3050 3200
 	0    -1   -1   0
@@
 F 2 "Resistors_SMD:R_0603" V 2980 3300 50  0001 C CNN
 F 3 "~" H 3050 3300 50  0001 C CNN
+F 4 "-" H 0   0   50  0001 C CNN "購入済み"
 	1    3050 3300
 	0    -1   -1   0
@@
 F 3 "~" H 3550 1250 50  0001 C CNN
 F 4 "1%" V 3450 1250 50  0000 C CNN "Tolerance"
+F 5 "d" H 0   0   50  0001 C CNN "購入済み"
 	1    3550 1250
 	1    0    0    -1
@@
 F 3 "~" H 3550 1750 50  0001 C CNN
 F 4 "1%" V 3450 1750 50  0000 C CNN "Tolerance"
+F 5 "d" H 0   0   50  0001 C CNN "購入済み"
 	1    3550 1750
 	1    0    0    -1
@@
 F 2 "Resistors_SMD:R_0603" V 4230 1900 50  0001 C CNN
 F 3 "~" H 4300 1900 50  0001 C CNN
+F 4 "-" H 0   0   50  0001 C CNN "購入済み"
 	1    4300 1900
 	0    -1   -1   0
@@
 F 2 "Resistors_SMD:R_0603" V 4230 2000 50  0001 C CNN
 F 3 "~" H 4300 2000 50  0001 C CNN
+F 4 "-" H 0   0   50  0001 C CNN "購入済み"
 	1    4300 2000
 	0    -1   -1   0
@@
 F 2 "Resistors_SMD:R_0603" V 7580 1300 50  0001 C CNN
 F 3 "~" H 7650 1300 50  0001 C CNN
+F 4 "-" H 0   0   50  0001 C CNN "購入済み"
 	1    7650 1300
 	1    0    0    -1
@@
 F 2 "Capacitors_SMD:C_0402_NoSilk" H 4450 1400 50  0001 C CNN
 F 3 "~" H 4450 1400 50  0001 C CNN
+F 4 "d" H 0   0   50  0001 C CNN "購入済み"
 	1    4450 1400
 	1    0    0    -1
@@
 Wire Wire Line
 	6550 2200 7150 2200
-Text GLabel 7250 2000 2    50   Input ~ 0
+Text GLabel 7250 2000 2    50   Output ~ 0
 VBUS_0.5A
-Text GLabel 7250 2100 2    50   Input ~ 0
+Text GLabel 7250 2100 2    50   Output ~ 0
 VBUS_1.5A
-Text GLabel 7250 2200 2    50   Input ~ 0
+Text GLabel 7250 2200 2    50   Output ~ 0
 VBUS_3.0A
 $Comp
@@
 F 2 "Resistors_SMD:R_0603" V 6980 1700 50  0001 C CNN
 F 3 "~" H 7050 1700 50  0001 C CNN
+F 4 "-" H 0   0   50  0001 C CNN "購入済み"
 	1    7050 1700
 	1    0    0    1
@@
 F 2 "Resistors_SMD:R_0603" V 6880 1700 50  0001 C CNN
 F 3 "~" H 6950 1700 50  0001 C CNN
+F 4 "-" H 0   0   50  0001 C CNN "購入済み"
 	1    6950 1700
 	1    0    0    1
@@
 F 2 "Resistors_SMD:R_0603" V 7080 1700 50  0001 C CNN
 F 3 "~" H 7150 1700 50  0001 C CNN
+F 4 "-" H 0   0   50  0001 C CNN "購入済み"
 	1    7150 1700
 	1    0    0    1
@@
 Wire Wire Line
 	7150 2200 7250 2200
-$Comp
-L power:+3V3 #PWR0129
-U 1 1 5BB6ECC3
-P 6950 1300
-F 0 "#PWR0129" H 6950 1150 50  0001 C CNN
-F 1 "+3V3" H 6950 1440 50  0000 C CNN
-F 2 "" H 6950 1300 50  0001 C CNN
-F 3 "" H 6950 1300 50  0001 C CNN
-	1    6950 1300
-	1    0    0    -1
-$EndComp
 Wire Wire Line
 	6950 1550 6950 1350
@@
 F 2 "Connectors_JST:JST_XH_S05B-XH-A_05x2.50mm_Angled" H 10100 1200 50  0001 C CNN
 F 3 "~" H 10100 1200 50  0001 C CNN
+F 4 "a" H 0   0   50  0001 C CNN "購入済み"
 	1    10100 1200
 	1    0    0    -1
 $EndComp
 Wire Wire Line
-	9650 1200 9800 1200
-Wire Wire Line
-	9900 1100 9800 1100
-Wire Wire Line
-	9800 1100 9800 1200
-Wire Wire Line
-	9800 1200 9900 1200
-Connection ~ 9800 1200
+	9650 1400 9800 1400
+Wire Wire Line
+	9900 1300 9800 1300
+Wire Wire Line
+	9800 1300 9800 1400
+Wire Wire Line
+	9800 1400 9900 1400
+Connection ~ 9800 1400
 $Comp
 L power:GND #PWR0130
 U 1 1 5BB7A1A5
-P 9800 1450
-F 0 "#PWR0130" H 9800 1200 50  0001 C CNN
-F 1 "GND" H 9800 1300 50  0000 C CNN
-F 2 "" H 9800 1450 50  0001 C CNN
-F 3 "" H 9800 1450 50  0001 C CNN
-	1    9800 1450
-	1    0    0    -1
-$EndComp
-Wire Wire Line
-	9900 1300 9800 1300
-Wire Wire Line
-	9800 1300 9800 1400
-Wire Wire Line
-	9900 1400 9800 1400
-Wire Wire Line
-	9800 1400 9800 1450
-Connection ~ 9800 1400
-Text GLabel 9650 1200 0    50   Output ~ 0
+P 9250 1250
+F 0 "#PWR0130" H 9250 1000 50  0001 C CNN
+F 1 "GND" H 9250 1100 50  0000 C CNN
+F 2 "" H 9250 1250 50  0001 C CNN
+F 3 "" H 9250 1250 50  0001 C CNN
+	1    9250 1250
+	1    0    0    -1
+$EndComp
+Wire Wire Line
+	9900 1100 9250 1100
+Wire Wire Line
+	9250 1100 9250 1200
+Wire Wire Line
+	9900 1200 9250 1200
+Wire Wire Line
+	9250 1200 9250 1250
+Connection ~ 9250 1200
+Text GLabel 9650 1400 0    50   Output ~ 0
 VIN
 Wire Wire Line
@@
 F 2 "Housings_QFP:LQFP-48_7x7mm_Pitch0.5mm" H 8400 4700 60  0001 C CNN
 F 3 "" H 8400 4700 60  0000 C CNN
+F 4 "a" H 0   0   50  0001 C CNN "購入済み"
 	1    8400 4700
 	1    0    0    -1
@@
 F 2 "KiCad_Footprints:DSC1001_CDFN-4_3.2x2.5" H 6150 6300 60  0001 C CNN
 F 3 "" H 6150 6300 60  0001 C CNN
+F 4 "d" H 0   0   50  0001 C CNN "購入済み"
 	1    6150 6300
 	1    0    0    -1
@@
 F 2 "Capacitors_SMD:C_0402_NoSilk" H 5000 6150 50  0001 C CNN
 F 3 "~" H 5000 6150 50  0001 C CNN
+F 4 "-" H 0   0   50  0001 C CNN "購入済み"
 	1    5000 6150
 	1    0    0    -1
@@
 F 2 "TO_SOT_Packages_SMD:SOT-23-6" H 5450 5100 60  0001 C CNN
 F 3 "" H 5450 5100 60  0001 C CNN
+F 4 "d" H 0   0   50  0001 C CNN "購入済み"
 	1    5450 5100
 	1    0    0    -1
@@
 F 2 "Capacitors_SMD:C_0402_NoSilk" H 4850 5050 50  0001 C CNN
 F 3 "~" H 4850 5050 50  0001 C CNN
+F 4 "-" H 0   0   50  0001 C CNN "購入済み"
 	1    4850 5050
 	1    0    0    -1
@@
 F 2 "Resistors_SMD:R_0603" V 6080 5200 50  0001 C CNN
 F 3 "~" H 6150 5200 50  0001 C CNN
+F 4 "-" H 0   0   50  0001 C CNN "購入済み"
 	1    6150 5200
 	0    -1   -1   0
@@
 F 2 "Resistors_SMD:R_0603" V 5880 4700 50  0001 C CNN
 F 3 "~" H 5950 4700 50  0001 C CNN
+F 4 "-" H 0   0   50  0001 C CNN "購入済み"
 	1    5950 4700
 	1    0    0    -1
@@
 F 3 "~" H 7200 4700 50  0001 C CNN
 F 4 "1%" V 7100 4700 50  0000 C CNN "Tolerance"
+F 5 "d" H 0   0   50  0001 C CNN "購入済み"
 	1    7200 4700
 	0    -1   -1   0
@@
 F 2 "Capacitors_SMD:C_0402_NoSilk" H 7200 3850 50  0001 C CNN
 F 3 "~" H 7200 3850 50  0001 C CNN
+F 4 "-" H 0   0   50  0001 C CNN "購入済み"
 	1    7200 3850
 	1    0    0    -1
@@
 F 2 "Capacitors_SMD:C_0402_NoSilk" H 6950 3800 50  0001 C CNN
 F 3 "~" H 6950 3800 50  0001 C CNN
+F 4 "-" H 0   0   50  0001 C CNN "購入済み"
 	1    6950 3800
 	1    0    0    -1
@@
 F 2 "Capacitors_SMD:C_0402_NoSilk" H 6650 3700 50  0001 C CNN
 F 3 "~" H 6650 3700 50  0001 C CNN
+F 4 "-" H 0   0   50  0001 C CNN "購入済み"
 	1    6650 3700
 	1    0    0    -1
@@
 F 2 "Capacitors_SMD:C_0603" H 6400 3700 50  0001 C CNN
 F 3 "~" H 6400 3700 50  0001 C CNN
+F 4 "a" H 0   0   50  0001 C CNN "購入済み"
 	1    6400 3700
 	1    0    0    -1
@@
 F 2 "Capacitors_SMD:C_0402_NoSilk" H 2850 5050 50  0001 C CNN
 F 3 "~" H 2850 5050 50  0001 C CNN
+F 4 "-" H 0   0   50  0001 C CNN "購入済み"
 	1    2850 5050
 	1    0    0    -1
@@
 F 2 "Capacitors_SMD:C_0603" H 2600 5050 50  0001 C CNN
 F 3 "~" H 2600 5050 50  0001 C CNN
+F 4 "a" H 0   0   50  0001 C CNN "購入済み"
 	1    2600 5050
 	1    0    0    -1
@@
 F 2 "LEDs:LED_0603" H 2600 2200 50  0001 C CNN
 F 3 "~" H 2600 2200 50  0001 C CNN
+F 4 "-" H 0   0   50  0001 C CNN "購入済み"
 	1    2600 2200
 	0    1    1    0
@@
 F 2 "LEDs:LED_0603" H 2750 2200 50  0001 C CNN
 F 3 "~" H 2750 2200 50  0001 C CNN
+F 4 "-" H 0   0   50  0001 C CNN "購入済み"
 	1    2750 2200
 	0    1    1    0
@@
 F 2 "Capacitors_SMD:C_0402_NoSilk" H 8800 2850 50  0001 C CNN
 F 3 "~" H 8800 2850 50  0001 C CNN
+F 4 "-" H 0   0   50  0001 C CNN "購入済み"
 	1    8800 2850
 	1    0    0    -1
@@
 F 2 "Capacitors_SMD:C_0402_NoSilk" H 9050 2850 50  0001 C CNN
 F 3 "~" H 9050 2850 50  0001 C CNN
+F 4 "-" H 0   0   50  0001 C CNN "購入済み"
 	1    9050 2850
 	1    0    0    -1
@@
 F 2 "Capacitors_SMD:C_0402_NoSilk" H 9300 2850 50  0001 C CNN
 F 3 "~" H 9300 2850 50  0001 C CNN
+F 4 "-" H 0   0   50  0001 C CNN "購入済み"
 	1    9300 2850
 	1    0    0    -1
@@
 F 0 "L7" V 3075 6350 50  0000 L CNN
 F 1 "600ohm@100MHz" V 2900 6300 50  0000 C CNN
-F 2 "Inductors_SMD:L_0603" V 2930 6300 50  0001 C CNN
+F 2 "Inductors_SMD:L_0402" V 2930 6300 50  0001 C CNN
 F 3 "~" H 3000 6300 50  0001 C CNN
+F 4 "d" H 0   0   50  0001 C CNN "購入済み"
 	1    3000 6300
 	0    -1   -1   0
@@
 F 2 "Capacitors_SMD:C_0402_NoSilk" H 3500 6450 50  0001 C CNN
 F 3 "~" H 3500 6450 50  0001 C CNN
+F 4 "-" H 0   0   50  0001 C CNN "購入済み"
 	1    3500 6450
 	1    0    0    -1
@@
 F 0 "L6" V 3075 5850 50  0000 L CNN
 F 1 "600ohm@100MHz" V 2900 5800 50  0000 C CNN
-F 2 "Inductors_SMD:L_0603" V 2930 5800 50  0001 C CNN
+F 2 "Inductors_SMD:L_0402" V 2930 5800 50  0001 C CNN
 F 3 "~" H 3000 5800 50  0001 C CNN
+F 4 "d" H 0   0   50  0001 C CNN "購入済み"
 	1    3000 5800
 	0    -1   -1   0
@@
 F 2 "Capacitors_SMD:C_0402_NoSilk" H 3500 5950 50  0001 C CNN
 F 3 "~" H 3500 5950 50  0001 C CNN
+F 4 "-" H 0   0   50  0001 C CNN "購入済み"
 	1    3500 5950
 	1    0    0    -1
@@
 F 2 "Resistors_SMD:R_0603" V 3180 7300 50  0001 C CNN
 F 3 "~" H 3250 7300 50  0001 C CNN
+F 4 "-" H 0   0   50  0001 C CNN "購入済み"
 	1    3250 7300
 	1    0    0    -1
@@
 Wire Wire Line
 	8150 1000 9900 1000
+$Comp
+L power:+1V8 #PWR0118
+U 1 1 5B9DDDE3
+P 6950 1300
+F 0 "#PWR0118" H 6950 1150 50  0001 C CNN
+F 1 "+1V8" H 6950 1440 50  0000 C CNN
+F 2 "" H 6950 1300 50  0001 C CNN
+F 3 "" H 6950 1300 50  0001 C CNN
+	1    6950 1300
+	1    0    0    -1
+$EndComp
 $EndSCHEMATC
