File: ZynqBoard/PCB/ZynqBoard/ZynqPower.sch (KiCad schematic (older format))
At the start: 60 parts, among them U1 XC7Z020-1CLG484C

Commit message: ZynqBoard PCB 設計完了
Parts:
- C24, C35, C36, C42, C43, C48, C49, C52, C59, C60, C72, C81, U1: 購入済み (none) -> d
- C25, C26, C27, C28, C29, C30, C31, C32, C33, C34, C37, C38, C39, C40, C41, C44, C45, C46, C47, C50, C51, C53, C54, C55, C56, C57, C58, C61, C62, C63, C64, C65, C66, C67, C68, C69, C70, C71, C73, C74, C75, C76, C77, C79, C80: 購入済み (none) -> a
- C78: footprint Capacitors_SMD:C_0603 -> Capacitors_SMD:C_0402_NoSilk; 購入済み (none) -> a
- L1: footprint Inductors_SMD:L_0603 -> Inductors_SMD:L_0402; 購入済み (none) -> d
